File: Bus_Board.kicad_pcb (KiCad board)
At the start: 2 copper layers, 295.9 x 39.4 mm, 44 parts, among them J1 +5V, J10 Conn_02x05_Odd_Even, J11 Conn_02x08_Odd_Even, J12 Conn_02x05_Odd_Even, J13 Conn_02x08_Odd_Even, J14 Conn_02x05_Odd_Even, J15 Conn_02x08_Odd_Even, J16 Conn_02x05_Odd_Even, J17 Conn_02x08_Odd_Even, J18 Conn_02x05_Odd_Even, J19 Conn_02x08_Odd_Even, J2 +12V, J20 Conn_02x05_Odd_Even, J21 Conn_02x08_Odd_Even, J22 Conn_02x05_Odd_Even, J23 Conn_02x08_Odd_Even, J24 Conn_02x05_Odd_Even, J25 +5V, J26 +12V, J27 GND, J28 -12V, J3 GND, J4 -12V, J5 Conn_02x08_Odd_Even, J6 Conn_02x05_Odd_Even, J7 Conn_02x08_Odd_Even, J8 Conn_02x05_Odd_Even, J9 Conn_02x08_Odd_Even

Commit message: Change text on PCB
Other:
- board text added: "EURORACK BUS BOARD V0.2.0"
- board text removed: "BUS BOARD V0.2.0"
Changed lines of the file:
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@@
     (effects (font (size 1 1) (thickness 0.15)))
   )
-  (gr_text "BUS BOARD V0.2.0" (at -113.665 50.165) (layer "F.SilkS")
+  (gr_text "EURORACK BUS BOARD V0.2.0" (at -109.22 50.165) (layer "F.SilkS")
     (effects (font (size 1 1) (thickness 0.15)))
   )
